File: m4dl/main.sch (KiCad schematic (older format))
At the start: 105 parts, among them IC1 NCP380, IC2 STM32F405RxTx, IC3 MCP2562, IC4 LTC2983, J1 TEMP2-8, J2 PRESSURE, J3 WEST TOP, J4 EAST TOP, J5 TEMP1, J6 TEMP9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

Commit message: Streamlined dl
Parts:
- removed C20, C21: 1n, Capacitors_SMD:C_0603, symbol pressure-rescue:C_Small
- removed C28, C37: 1n, Capacitors_SMD:C_0603, symbol temperature-rescue:C_Small
- removed D1: LED, agg:0603-LED, symbol main-rescue:LED
- removed D11: D, Diodes_SMD:SOD-123, symbol temperature-rescue:D
- removed D8, D9: ESD_DIODE, agg:0402, symbol pressure-rescue:ESD_DIODE
- removed IC4: LTC2983, agg:LQFP-48, symbol temperature-rescue:LTC2983
- removed J5: TEMP1, Connectors_Molex:Connector_Molex_PicoBlade_53048-0210, symbol temperature-rescue:CONN_01x02
- removed J6: TEMP9, Connectors_Molex:Connector_Molex_PicoBlade_53048-0210, symbol temperature-rescue:CONN_01x02
- removed R1: 1k, agg:0603-L, symbol main-rescue:R
- removed R14, R15: 3.74K, Resistors_SMD:R_0603, symbol pressure-rescue:R
- removed R23, R28, R33, R37: 3.74K, Resistors_SMD:R_0603, symbol temperature-rescue:R
- added IC?: LTC2986, agg:LQFP-48, symbol temperature-rescue:LTC2986
- R7: Farnell 2309108 -> 2073354
Connections:
- net TEMP8+ is gone; now on net TEMP7+: J1.2
- net TEMP8- is gone; now on net TEMP7-: J1.1
- net 3v3: now also IC?.2 (VDD), IC?.4 (VDD), IC?.45 (VDD), IC?.6 (VDD), IC?.8 (VDD)
- net CH1+: now also IC?.16 (CH1)
- net CH2+: now also IC?.17 (CH2)
- net CH3+: now also IC?.18 (CH3)
- net CH4+: now also IC?.19 (CH4)
- net CH5+: now also IC?.20 (CH5)
- net CH6+: now also IC?.21 (CH6)
- net CH7+: now also IC?.22 (CH7)
- net GND: now also IC?.1 (GND), IC?.12 (GND), IC?.15 (GND), IC?.3 (GND), IC?.36 (CH_GND), IC?.44 (GND), IC?.5 (GND), IC?.7 (GND), IC?.9 (GND)
- net SPI1_CS: now also IC?.41 (~CS)
- net SPI1_MISO: now also IC?.39 (SDO)
- net SPI1_MOSI: now also IC?.40 (SDI)
- net SPI1_SCK: now also IC?.38 (SCK)
- net TEMP1+: now also J1.14
- net TEMP1-: now also J1.13
- net TEMP2+: now also J1.12; no longer J1.14
- net TEMP2-: now also J1.11; no longer J1.13
- net TEMP3+: now also J1.10; no longer J1.12
- net TEMP3-: now also J1.9; no longer J1.11
- net TEMP4+: now also J1.8; no longer J1.10
- net TEMP4-: now also J1.7; no longer J1.9
- net TEMP5+: now also J1.6; no longer J1.8
- net TEMP5-: now also J1.5; no longer J1.7
- net TEMP6+: now also J1.4; no longer J1.6
- net TEMP6-: now also J1.3; no longer J1.5
- net TEMP7+: no longer J1.4
- net TEMP7-: no longer J1.3
- net TEMP_INT: now also IC?.37 (INT)
- net at C33.2: now also IC?.43 (LDO)
- net at C31.2: now also IC?.13 (VREF_OUT), IC?.14 (VREF_P)
- net at C32.2: now also IC?.11 (VREF_BYP)
- net at R29.2: now also IC?.42 (~RESET)
- net at C29.1: now also IC?.46 (Q3)
- net at C23.2: now also IC?.47 (Q2)
- net at C23.1: now also IC?.48 (Q1)
- net P4+: no longer names the net of J2.6
- net P5+: no longer names the net of J2.7
- net PRESSURE4: no longer names the net of IC2.24 (PC4)
- net PRESSURE5: no longer names the net of IC2.25 (PC5)
- no-connect marks 41 -> 40
Other:
- note added: "LTC2986:"
- note removed: "LTC2983:"
- moved on the sheet: C25, C26, C27, C35, C36, R20, R21, R22, R25, R26, R27, R31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
