File: m4dl/m4dl.sch (KiCad schematic (older format))
At the start: 91 parts

Commit message: Reorganise dl
Parts:
- removed C?: 10u, Capacitors_SMD:C_0603, symbol cusf-kicad:C
- removed C?: 1u, agg:0402-L, symbol cusf-kicad:C
- removed C? (x2): 1n, symbol cusf-kicad:C
- removed D? (x2): ESD_DIODE, agg:0402, symbol cusf-kicad:ESD_DIODE
- removed IC?: LTC2986, agg:LQFP-48, symbol cusf-kicad:LTC2986
- removed R? (x12): 3k74, symbol cusf-kicad:R
- added C? (x2): 1n, symbol cusf-kicad:C
- added C?: 10u, Capacitors_SMD:C_0603, symbol cusf-kicad:C
- added D? (x2): ESD_DIODE, agg:0402, symbol cusf-kicad:ESD_DIODE
- added IC?: LTC2986, agg:LQFP-48, symbol cusf-kicad:LTC2986
- added R? (x12): 3k74, symbol cusf-kicad:R
Connections:
- net 3v3: now also C?.1, IC?.2 (VDD), IC?.4 (VDD), IC?.45 (VDD), IC?.6 (VDD), IC?.8 (VDD); no longer C?.2
- net CH1+: now also IC?.16 (CH1), R?.1
- net CH2+: now also IC?.17 (CH2)
- net CH3+: now also IC?.18 (CH3), R?.1
- net CH4+: now also IC?.19 (CH4), R?.1
- net CH5+: now also IC?.20 (CH5), R?.1
- net CH6+: now also IC?.21 (CH6), R?.1
- net CH7+: now also IC?.22 (CH7), R?.1
- net GND: now also C?.2, C?.1, C?.2, C?.2, D?.1, D?.1, IC?.1 (GND), IC?.12 (GND), IC?.15 (GND), IC?.26 (GND), IC?.27 (GND), IC?.28 (GND), IC?.29 (GND), IC?.3 (GND), IC?.30 (GND), IC?.31 (GND), IC?.32 (GND), IC?.33 (GND), IC?.34 (GND), IC?.35 (GND), IC?.36 (COM), IC?.44 (GND), IC?.5 (GND), IC?.7 (GND), IC?.9 (GND), R?.1, R?.1, R?.1, R?.1, R?.1, R?.1; no longer C?.1, J?.8
- net P1+: now also D?.2
- net P2+: now also D?.2
- net PRESSURE1: now also C?.1
- net PRESSURE2: now also C?.1
- net SPI1_CS: now also IC?.41 (~CS)
- net SPI1_MISO: now also IC?.39 (SDA)
- net SPI1_MOSI: now also IC?.40 (SDI)
- net SPI1_SCK: now also IC?.38 (SCK)
- net TEMP1+: now also R?.2
- net TEMP1-: now also R?.2
- net TEMP3+: now also R?.2
- net TEMP3-: now also R?.2
- net TEMP4+: now also R?.2
- net TEMP4-: now also R?.2
- net TEMP5+: now also R?.2
- net TEMP5-: now also R?.2
- net TEMP6+: now also R?.2
- net TEMP6-: now also R?.2
- net TEMP7+: now also R?.2
- net TEMP7-: now also R?.2
- net TEMP_INT: now also IC?.37 (INT)
- net at C?.1: now also IC?.46 (Q3)
- net at C?.2: now also IC?.11 (VREF_BYP)
- net at C?.2: now also IC?.13 (VREF_OUT), IC?.14 (VREF_P)
- net at R?.2: now also IC?.42 (~RESET)
- net at C?.2: now also IC?.47 (Q2)
- net at C?.1: now also IC?.48 (Q1)
- new net: C?.2, IC?.43 (LDO)
- no-connect marks 54 -> 55
Other:
- note added: "Current Limiting"
- note added: "GLOBAL INTERCONNECTS"
- note added: "MICRO SD CARD"
- note added: "MICROCONTROLLER"
- note added: "PRESSURE FILTERS"
- note added: "SENSOR INTERCONNECTS"
- note added: "TEMPERATURE FILTERS"
- note added: "TEMPERATURE MEASUREMENT"
- note added: "UART"
- note added: "USB"
- note removed: "CURRENT LIMITING:"
- note removed: "FILTERS:"
- note removed: "GLOBAL INTERCONNECTS:"
- note removed: "LTC2986:"
- note removed: "MAIN"
- note removed: "MCU Peripherals:"
- note removed: "PRESSURE"
- note removed: "STM32F405:"
- note removed: "TEMPERATURE"
- moved on the sheet: C?, D?, IC?, J?, P?, R?, U?, Y?
