File: m4pyro/m4pyro.sch (KiCad schematic (older format))
At the start: 75 parts, among them IC1 MCP2562, J1 WEST TOP, J2 EAST TOP, P1 SWD_TC, Y1 26M

Commit message: Use cusf-kicad.lib instead of agg-kicad.lib
Parts:
- C1, C10, C11, C12, C13, C2, C3, C4, C5, C6, C7, C8, C9: symbol agg-kicad:C -> cusf-kicad:C
- D1, D2, D3: symbol agg-kicad:LED -> cusf-kicad:LED
- D? (x3): symbol agg-kicad:D -> cusf-kicad:D
- D? (x3): symbol agg-kicad:SCHOTTKY -> cusf-kicad:SCHOTTKY
- IC1: symbol agg-kicad:MCP2562 -> cusf-kicad:MCP2562
- IC? (x3): symbol agg-kicad:LTC4151 -> cusf-kicad:LTC4151
- IC?: symbol agg-kicad:STM32F405RxTx -> cusf-kicad:STM32F405RxTx
- J1, J2: symbol agg-kicad:CONN_02x15 -> cusf-kicad:CONN_02x15
- J? (x3): symbol agg-kicad:CONN_01x04 -> cusf-kicad:CONN_01x04
- K? (x3): symbol agg-kicad:RELAY_SPST -> cusf-kicad:RELAY_SPST
- P1: symbol agg-kicad:SWD_TC -> cusf-kicad:SWD_TC
- Q? (x3): symbol agg-kicad:NFET -> cusf-kicad:NFET
- R108, R3, R5, R6, R7, R? (x21): symbol agg-kicad:R -> cusf-kicad:R
- X? (x9): symbol agg-kicad:PART -> cusf-kicad:PART
- Y1: symbol agg-kicad:SMD_XTAL -> cusf-kicad:SMD_XTAL
