File: m4_board_template/m4_board_template.sch (KiCad schematic (older format))
At the start: 27 parts, among them IC1 MCP2562, IC2 STM32F405RxTx, J1 WEST TOP, J2 EAST TOP, P1 SWD_TC, Y1 26M

Commit message: Use cusf-kicad.lib instead of agg-kicad.lib
Parts:
- C1, C10, C11, C12, C13, C2, C3, C4, C5, C6, C7, C8, C9: symbol agg-kicad:C -> cusf-kicad:C
- D1, D2, D3: symbol agg-kicad:LED -> cusf-kicad:LED
- IC1: symbol agg-kicad:MCP2562 -> cusf-kicad:MCP2562
- IC2: symbol agg-kicad:STM32F405RxTx -> cusf-kicad:STM32F405RxTx
- J1, J2: symbol agg-kicad:CONN_02x15 -> cusf-kicad:CONN_02x15
- P1: symbol agg-kicad:SWD_TC -> cusf-kicad:SWD_TC
- R108, R3, R5, R6, R7: symbol agg-kicad:R -> cusf-kicad:R
- Y1: symbol agg-kicad:SMD_XTAL -> cusf-kicad:SMD_XTAL
Changed lines of the file:
@@
 $EndDescr
 $Comp
-L agg-kicad:MCP2562 IC1
+L cusf-kicad:MCP2562 IC1
 U 1 1 5AA4FF08
 P 1850 9200
@@
 $EndComp
 $Comp
-L agg-kicad:3v3 #PWR06
+L cusf-kicad:3v3 #PWR06
 U 1 1 5AA4FF0F
 P 1400 8950
@@
 5v_CAN
 $Comp
-L agg-kicad:GND #PWR07
+L cusf-kicad:GND #PWR07
 U 1 1 5AA4FF16
 P 1400 9450
@@
 CAN_RXD
 $Comp
-L agg-kicad:C C3
+L cusf-kicad:C C3
 U 1 1 5AA4FF21
 P 1250 9150
@@
 $EndComp
 $Comp
-L agg-kicad:LED D1
+L cusf-kicad:LED D1
 U 1 1 5AA4FF29
 P 4050 8850
@@
 $EndComp
 $Comp
-L agg-kicad:R R5
+L cusf-kicad:R R5
 U 1 1 5AA4FF31
 P 3750 8850
@@
 $EndComp
 $Comp
-L agg-kicad:R R6
+L cusf-kicad:R R6
 U 1 1 5AA4FF39
 P 3750 9150
@@
 $EndComp
 $Comp
-L agg-kicad:R R7
+L cusf-kicad:R R7
 U 1 1 5AA4FF41
 P 3750 9450
@@
 $EndComp
 $Comp
-L agg-kicad:LED D2
+L cusf-kicad:LED D2
 U 1 1 5AA4FF49
 P 4050 9150
@@
 $EndComp
 $Comp
-L agg-kicad:LED D3
+L cusf-kicad:LED D3
 U 1 1 5AA4FF51
 P 4050 9450
@@
 $EndComp
 $Comp
-L agg-kicad:GND #PWR025
+L cusf-kicad:GND #PWR025
 U 1 1 5AA4FF58
 P 4150 8900
@@
 $EndComp
 $Comp
-L agg-kicad:GND #PWR026
+L cusf-kicad:GND #PWR026
 U 1 1 5AA4FF5E
 P 4150 9200
@@
 $EndComp
 $Comp
-L agg-kicad:GND #PWR027
+L cusf-kicad:GND #PWR027
 U 1 1 5AA4FF64
 P 4150 9500
@@
 	2850 4700 2950 4700
 $Comp
-L agg-kicad:PWR #FLG01
+L cusf-kicad:PWR #FLG01
 U 1 1 5AA4FFBF
 P 900 9100
@@
 	1800 4700 1800 4800
 $Comp
-L agg-kicad:GND #PWR02
+L cusf-kicad:GND #PWR02
 U 1 1 5AA4FFFD
 P 1250 1100
@@
 $EndComp
 $Comp
-L agg-kicad:GND #PWR013
+L cusf-kicad:GND #PWR013
 U 1 1 5AA50003
 P 1750 1100
@@
 	1350 1950 1250 1950
 $Comp
-L agg-kicad:CONN_02x15 J2
+L cusf-kicad:CONN_02x15 J2
 U 1 1 5AA50050
 P 3050 1150
@@
 UART_TX
 $Comp
-L agg-kicad:GND #PWR020
+L cusf-kicad:GND #PWR020
 U 1 1 5AA500B8
 P 2750 2650
@@
 $EndComp
 $Comp
-L agg-kicad:GND #PWR022
+L cusf-kicad:GND #PWR022
 U 1 1 5AA500BE
 P 3250 2650
@@
 $EndComp
 $Comp
-L agg-kicad:GND #PWR019
+L cusf-kicad:GND #PWR019
 U 1 1 5AA500C4
 P 2750 1100
@@
 Connection ~ 2750 1150
 $Comp
-L agg-kicad:GND #PWR021
+L cusf-kicad:GND #PWR021
 U 1 1 5AA500CE
 P 3250 1100
@@
 	3250 2550 3250 2450
 $Comp
-L agg-kicad:GND #PWR03
+L cusf-kicad:GND #PWR03
 U 1 1 5AA500F3
 P 1250 2650
@@
 	1250 2550 1250 2650
 $Comp
-L agg-kicad:GND #PWR014
+L cusf-kicad:GND #PWR014
 U 1 1 5AA500FE
 P 1750 2650
@@
 RSVD13
 $Comp
-L agg-kicad:SWD_TC P1
+L cusf-kicad:SWD_TC P1
 U 1 1 5AA50189
 P 2350 8000
@@
 $EndComp
 $Comp
-L agg-kicad:3v3 #PWR017
+L cusf-kicad:3v3 #PWR017
 U 1 1 5AA50190
 P 1900 7850
@@
 $EndComp
 $Comp
-L agg-kicad:GND #PWR018
+L cusf-kicad:GND #PWR018
 U 1 1 5AA50196
 P 1900 8150
@@
 	650  3350 4400 3350
 $Comp
-L agg-kicad:C C9
+L cusf-kicad:C C9
 U 1 1 5AA501AC
 P 1450 8050
@@
 $EndComp
 $Comp
-L agg-kicad:GND #PWR011
+L cusf-kicad:GND #PWR011
 U 1 1 5AA501B3
 P 1450 8150
@@
 	1450 8050 1450 8150
 $Comp
-L agg-kicad:3v3 #PWR010
+L cusf-kicad:3v3 #PWR010
 U 1 1 5AA501BA
 P 1450 7850
@@
 PB4 is JTRST, DO NOT CONNECT (Errata 2.1.4)
 $Comp
-L agg-kicad:SMD_XTAL Y1
+L cusf-kicad:SMD_XTAL Y1
 U 1 1 5AA501C3
 P 1500 5550
@@
 $EndComp
 $Comp
-L agg-kicad:C C1
+L cusf-kicad:C C1
 U 1 1 5AA501CB
 P 1200 5400
@@
 $EndComp
 $Comp
-L agg-kicad:GND #PWR01
+L cusf-kicad:GND #PWR01
 U 1 1 5AA501D2
 P 1050 5600
@@
 Connection ~ 1500 5800
 $Comp
-L agg-kicad:R R3
+L cusf-kicad:R R3
 U 1 1 5AA501EA
 P 1700 5700
@@
 	1500 5800 1650 5800
 $Comp
-L agg-kicad:C C2
+L cusf-kicad:C C2
 U 1 1 5AA501FC
 P 1200 5800
@@
 $EndComp
 $Comp
-L agg-kicad:C C10
+L cusf-kicad:C C10
 U 1 1 5AA50204
 P 1550 3900
@@
 $EndComp
 $Comp
-L agg-kicad:C C7
+L cusf-kicad:C C7
 U 1 1 5AA5020C
 P 1350 4400
@@
 $EndComp
 $Comp
-L agg-kicad:C C4
+L cusf-kicad:C C4
 U 1 1 5AA50214
 P 1350 3800
@@
 $EndComp
 $Comp
-L agg-kicad:C C5
+L cusf-kicad:C C5
 U 1 1 5AA5021C
 P 1350 4000
@@
 $EndComp
 $Comp
-L agg-kicad:C C11
+L cusf-kicad:C C11
 U 1 1 5AA50224
 P 1550 4100
@@
 $EndComp
 $Comp
-L agg-kicad:C C6
+L cusf-kicad:C C6
 U 1 1 5AA5022C
 P 1350 4200
@@
 $EndComp
 $Comp
-L agg-kicad:C C8
+L cusf-kicad:C C8
 U 1 1 5AA50234
 P 1450 4300
@@
 	1300 4400 1300 4500
 $Comp
-L agg-kicad:C C13
+L cusf-kicad:C C13
 U 1 1 5AA5025B
 P 1750 5000
@@
 	1850 5100 1600 5100
 $Comp
-L agg-kicad:C C12
+L cusf-kicad:C C12
 U 1 1 5AA50267
 P 1600 5100
@@
 $EndComp
 $Comp
-L agg-kicad:GND #PWR08
+L cusf-kicad:GND #PWR08
 U 1 1 5AA5026E
 P 1450 5000
@@
 $EndComp
 $Comp
-L agg-kicad:GND #PWR09
+L cusf-kicad:GND #PWR09
 U 1 1 5AA50274
 P 1450 5100
@@
 	650  800  650  2950
 $Comp
-L agg-kicad:PWR #FLG02
+L cusf-kicad:PWR #FLG02
 U 1 1 5AAEFC0F
 P 2700 2550
@@
 	2850 5900 2950 5900
 $Comp
-L agg-kicad:CONN_02x15 J1
+L cusf-kicad:CONN_02x15 J1
 U 1 1 5AA50022
 P 1550 1150
@@
 NoConn ~ 2850 1650
 $Comp
-L agg-kicad:R R108
+L cusf-kicad:R R108
 U 1 1 5A9B48C6
 P 2350 9650
@@
 3v3_MOTOR
 $Comp
-L agg-kicad:STM32F405RxTx IC2
+L cusf-kicad:STM32F405RxTx IC2
 U 1 1 5AA4FFC6
 P 2350 5700
@@
 NoConn ~ 2850 4300
 $Comp
-L agg-kicad:GND #PWR?
+L cusf-kicad:GND #PWR?
 U 1 1 5E8266D0
 P 1800 5400
@@
 $EndComp
 $Comp
-L agg-kicad:GND #PWR?
+L cusf-kicad:GND #PWR?
 U 1 1 5E833C33
 P 1700 4800
@@
 $EndComp
 $Comp
-L agg-kicad:GND #PWR?
+L cusf-kicad:GND #PWR?
 U 1 1 5E833CF7
 P 1300 4500
@@
 $EndComp
 $Comp
-L agg-kicad:3v3 #PWR?
+L cusf-kicad:3v3 #PWR?
 U 1 1 5E84101C
 P 1800 3850
