File: m4fc/m4fc.sch (KiCad schematic (older format))
At the start: 39 parts, among them IC1 MCP2562, IC2 STM32F405RxTx, IC3 MS5540C, IC4 ADXL345, J1 WEST TOP, J2 EAST TOP, P1 SWD_TC, Q1 NFET, X1 SG-3030CM, Y1 26M

Commit message: Use cusf-kicad.lib instead of agg-kicad.lib
Parts:
- C1, C10, C11, C12, C13, C14, C15, C16, C17, C18, C2, C3, C4, C5, C6, C7, C8, C9: symbol agg-kicad:C -> cusf-kicad:C
- D1, D2, D3: symbol agg-kicad:LED -> cusf-kicad:LED
- D4: symbol agg-kicad:D -> cusf-kicad:D
- IC1: symbol agg-kicad:MCP2562 -> cusf-kicad:MCP2562
- IC2: symbol agg-kicad:STM32F405RxTx -> cusf-kicad:STM32F405RxTx
- IC3: symbol agg-kicad:MS5540C -> cusf-kicad:MS5540C
- IC4: symbol agg-kicad:ADXL345 -> cusf-kicad:ADXL345
- J1, J2: symbol agg-kicad:CONN_02x15 -> cusf-kicad:CONN_02x15
- LS1: symbol agg-kicad:SOUNDER -> cusf-kicad:SOUNDER
- P1: symbol agg-kicad:SWD_TC -> cusf-kicad:SWD_TC
- Q1: symbol agg-kicad:NFET -> cusf-kicad:NFET
- R1, R2, R3, R4, R5, R6: symbol agg-kicad:R -> cusf-kicad:R
- Y1: symbol agg-kicad:SMD_XTAL -> cusf-kicad:SMD_XTAL
