File: m4fc/m4fc.sch (KiCad schematic (older format))
At the start: 39 parts, among them IC1 MCP2562, IC2 STM32F405RxTx, IC3 MS5540C, IC4 ADXL345, J1 WEST TOP, J2 EAST TOP, P1 SWD_TC, Q1 NFET, X1 SG-3030CM, Y1 26M

Commit message: Reorganise fc
Parts:
- removed C17, C18: 100n, agg:0402, symbol cusf-kicad:C
- added C? (x2): 100n, symbol cusf-kicad:C
- renumbered C15 to C?, C14 to C?, C16 to C?, C3 to C?, C9 to C?, C1 to C?, C2 to C?, C10 to C?, C7 to C?, C4 to C?, C5 to C?, C11 to C?, C6 to C?, C8 to C?, C13 to C?, C12 to C?, D4 to D?, D1 to D?, D2 to D?, D3 to D?, IC4 to IC?, IC1 to IC?, IC2 to IC?, IC3 to IC?, J1 to J?, J2 to J?, LS1 to LS?, P1 to P?, Q1 to Q?, R6 to R?, R2 to R?, R3 to R?, R4 to R?, R5 to R?, R1 to R?, X1 to X?, Y1 to Y?
Connections:
- net 3v3: now also IC?.5 (VDD), C?.1, C?.1; no longer IC?.4 (PEN)
- net BARO_DIN: now also IC?.7 (DIN)
- net BARO_SCLK: now also IC?.1 (SCLK); no longer IC?.2 (GND)
- net GND: now also IC?.2 (GND), X?.2 (GND), C?.2, C?.2
- net at IC?.3 (PV): no longer X?.3 (OUT)
- net at IC?.6 (MCLK): now also X?.3 (OUT)
Other:
- note added: "ACCELEROMETER"
- note added: "BAROMETER"
- note added: "BEEPER"
- moved on the sheet: C?, D?, IC?, LS?, Q?, R?, X?
