File: m4-avionics/m4dl.sch (KiCad schematic (older format))
At the start: 90 parts

Commit message: New global layout with hierarchical pins
Parts:
- removed C? (x4): 1n, symbol cusf-kicad:C
- removed D?: ESD_DIODE, agg:0402, symbol cusf-kicad:ESD_DIODE
- removed J?: PRESSURE, Connectors_Molex:Connector_Molex_PicoBlade_53048-1010, symbol cusf-kicad:CONN_02x05
- removed J?: TEMP2-8, Connectors_Molex:Connector_Molex_PicoBlade_53048-1410, symbol cusf-kicad:CONN_02x07
- removed J?: USB, Connectors_Molex:Connector_Molex_PicoBlade_53261-0471, symbol cusf-kicad:CONN_01x04
- removed J?: WEST TOP, agg:TFML-115-02-L-D-LC, symbol cusf-kicad:CONN_02x15
- removed J?: EAST TOP, agg:TFML-115-02-L-D-LC, symbol cusf-kicad:CONN_02x15
- removed J?: UART, symbol Connector_Generic:Conn_01x04
- removed R?: 1k, symbol cusf-kicad:R
- removed R? (x7): 3k74, symbol cusf-kicad:R
Connections:
- net labels added: 3V3, 5V_CAN
- net labels removed: 12v_DL, 3v3_AUX1, 3v3_AUX2, 3v3_DL, 3v3_FC, 3v3_MOTOR, 3v3_PYRO, 3v3_RADIO, 3v3_TOP, 5v_AUX1, 5v_AUX2, 5v_CAM1, 5v_CAM2, 5v_CAN, 5v_RADIO, CH5+, CH6+, CH7+, P3+, PRESSURE3, PWR, PYRO1, PYRO2, PYRO3, PYRO4, PYRO5, PYRO6, PYRO7, PYRO8, RSVD1, RSVD10, RSVD11, RSVD12, RSVD13, RSVD3, RSVD4, RSVD5, RSVD6, RSVD7, RSVD8, RSVD9, TEMP5+, TEMP5-, TEMP6+, TEMP6-, TEMP7+, TEMP7-
- wire segments 530 -> 379
- no-connect marks 55 -> 30
Other:
- note added: "PA2 (TX) <-> Pressure 1\nPA3 (RX) <-> Pressure 2"
- note added: "UART ISOLATOR"
- note removed: "GLOBAL INTERCONNECTS"
- note removed: "PA2(TX) <-> Pressure 1\nPA3 (RX) <-> Pressure 2"
- note removed: "SENSOR INTERCONNECTS"
- note removed: "UART"
- note removed: "USB"
- moved on the sheet: C?, D?, IC?, R?, U?
