File: m4-avionics/m4fc.sch (KiCad schematic (older format))
At the start: 40 parts

Commit message: New global layout with hierarchical pins
Parts:
- removed J?: WEST TOP, agg:TFML-115-02-L-D-LC, symbol cusf-kicad:CONN_02x15
- removed J?: EAST TOP, agg:TFML-115-02-L-D-LC, symbol cusf-kicad:CONN_02x15
Connections:
- net labels added: 3V3, 5V_CAN
- net labels removed: 12v_DL, 3v3_AUX1, 3v3_AUX2, 3v3_DL, 3v3_FC, 3v3_MOTOR, 3v3_PYRO, 3v3_RADIO, 3v3_TOP, 5v_AUX1, 5v_AUX2, 5v_CAM1, 5v_CAM2, 5v_CAN, 5v_RADIO, PWR, PYRO1, PYRO2, PYRO3, PYRO4, PYRO5, PYRO6, PYRO7, PYRO8, RSVD1, RSVD10, RSVD11, RSVD12, RSVD13, RSVD3, RSVD4, RSVD5, RSVD6, RSVD7, RSVD8, RSVD9, UART_RX, UART_TX
- wire segments 290 -> 222
- no-connect marks 26 -> 4
