File: schematics/dl/dl.sch (KiCad schematic (older format))
At the start: 62 parts

Commit message: Add sensor front-ends
Parts:
- removed C?: 1u, agg:0402-L, symbol cusf-kicad:C
- removed C? (x3): 10u, Capacitors_SMD:C_0603, symbol cusf-kicad:C
- removed C? (x6): 1n, symbol cusf-kicad:C
- removed C? (x2): 100n, Capacitors_SMD:C_0603, symbol cusf-kicad:C
- removed C?: 1u, Capacitors_SMD:C_0603, symbol cusf-kicad:C
- removed D? (x3): ESD_DIODE, agg:0402, symbol cusf-kicad:ESD_DIODE
- removed IC?: NCP380, agg:DFN-6-EP-ONSEMI, symbol cusf-kicad:NCP380
- removed IC?: LTC2986, agg:LQFP-48, symbol cusf-kicad:LTC2986
- removed R? (x4): 47k, symbol cusf-kicad:R
- removed R? (x10): 3k74, symbol cusf-kicad:R
- removed R?: 10k, symbol cusf-kicad:R
- removed R?: 110k, symbol cusf-kicad:R
- added C? (x10): 10n, symbol cusf-kicad:C
- added C? (x5): 1u, symbol cusf-kicad:C
- added C? (x4): 82n, symbol cusf-kicad:C
- added C? (x4): 8n2, symbol cusf-kicad:C
- added C? (x16): 100n, symbol cusf-kicad:C
- added D? (x8): ESD_DIODE, cusf:0402, symbol cusf-kicad:ESD_DIODE
- added IC?: ADP3335, cusf:MSOP-8, symbol cusf-kicad:ADP3335
- added IC? (x12): AD8656, cusf:MSOP-8, symbol cusf-kicad:AD8656
- added IC? (x4): AD8495, cusf:MSOP-8, symbol cusf-kicad:AD8495
- added R? (x6): 6k04, symbol cusf-kicad:R
- added R? (x4): 47k, symbol cusf-kicad:R
- added R? (x2): 562R, symbol cusf-kicad:R
- added R? (x2): 17k8, symbol cusf-kicad:R
- added R? (x12): 1k, symbol cusf-kicad:R
- added R? (x4): 8k87, symbol cusf-kicad:R
- added R? (x4): 31k6, symbol cusf-kicad:R
- added R? (x4): 2k94, symbol cusf-kicad:R
- added R? (x4): 95k3, symbol cusf-kicad:R
Connections:
- net labels added: 12V_DL, AGND, AVCC, P1, P2
- net labels removed: CH1+, CH2+, CH3+, CH4+, CH_GND, P1+, P2+
- wire segments 377 -> 613
- no-connect marks 28 -> 24
Other:
- note added: "- 150R current shunt required for\n 0.6v to 3v @ 4mA to 20mA\n\n- Pressure sensors are highest rate so\n should be connected to ADC123_x\n\n- All analog circuitry should be connected\n between VDD_A and AGND. AGND should\n be a separate sground plane connected to\n GND by a single trace wide enough to sink\n all of AGND"
- note added: "Analog Supply (500mA @ 3v3)"
- note added: "NOTES:"
- note added: "PRESSURE FRONT-ENDS"
- note added: "THERMOCOUPLE FRONT-ENDS"
- note removed: "Current Limiting"
- note removed: "PRESSURE FILTERS"
- note removed: "TEMPERATURE FILTERS"
- note removed: "TEMPERATURE MEASUREMENT"
- moved on the sheet: C?, D?, IC?, P?, R?, U?, Y?

Commit message: Fix pressure connectors
Connections:
- net labels added: P1+, P1-, P2+, P2-
- net labels removed: P1, P2
- wire segments 613 -> 615
Changed lines of the file:
@@
 OTG_HS_DP
 Text HLabel 13300 6800 0    50   Input ~ 0
-P1
-Text HLabel 13300 6900 0    50   Input ~ 0
-P2
-Wire Wire Line
-	13300 6900 13450 6900
+P1+
 Wire Wire Line
 	13450 6800 13300 6800
 Text Label 13450 6800 0    50   ~ 0
-P1
-Text Label 13450 6900 0    50   ~ 0
-P2
+P1+
 Text Label 1650 2800 2    50   ~ 0
 ~RST
@@
 	1    0    0    -1
 $EndComp
-Wire Wire Line
-	4800 9200 4800 8850
 Connection ~ 4800 9200
 Wire Wire Line
-	4800 8850 4600 8850
-Wire Wire Line
-	4800 8850 4800 8650
-Connection ~ 4800 8850
-$Comp
-L cusf-kicad:AVCC #PWR?
-U 1 1 60C8CBF9
-P 4800 8650
-F 0 "#PWR?" H 4800 8760 50  0001 L CNN
-F 1 "AVCC" H 4800 8750 50  0000 C CNN
-F 2 "" H 4800 8650 50  0001 C CNN
-F 3 "" H 4800 8650 50  0001 C CNN
-	1    4800 8650
-	1    0    0    -1
-$EndComp
-Text Label 4600 8850 0    50   ~ 0
-P1
-Wire Wire Line
 	6650 9100 6800 9100
 Wire Wire Line
@@
 	1    0    0    -1
 $EndComp
-Wire Wire Line
-	9650 9200 9650 8850
 Connection ~ 9650 9200
-Wire Wire Line
-	9650 8850 9450 8850
-Wire Wire Line
-	9650 8850 9650 8650
-Connection ~ 9650 8850
-$Comp
-L cusf-kicad:AVCC #PWR?
-U 1 1 60FAF464
-P 9650 8650
-F 0 "#PWR?" H 9650 8760 50  0001 L CNN
-F 1 "AVCC" H 9650 8750 50  0000 C CNN
-F 2 "" H 9650 8650 50  0001 C CNN
-F 3 "" H 9650 8650 50  0001 C CNN
-	1    9650 8650
-	1    0    0    -1
-$EndComp
-Text Label 9450 8850 0    50   ~ 0
-P2
 $Comp
 L cusf-kicad:R R?
@@
 	4400 8400 4400 9850
 Wire Notes Line
-	4400 9850 13850 9850
+	4400 9850 14300 9850
 Wire Notes Line
-	13850 9850 13850 8400
+	14300 9850 14300 8400
 Wire Notes Line
-	4400 8400 13850 8400
+	4400 8400 14300 8400
+Text Label 4600 9200 0    50   ~ 0
+P1-
+Text Label 9450 9200 0    50   ~ 0
+P2-
+Wire Wire Line
+	9450 9200 9650 9200
+Wire Wire Line
+	4600 9200 4800 9200
+Text HLabel 13300 6900 0    50   Input ~ 0
+P1-
+Wire Wire Line
+	13450 6900 13300 6900
+Text Label 13450 6900 0    50   ~ 0
+P1-
+Text HLabel 13300 7050 0    50   Input ~ 0
+P2+
+Wire Wire Line
+	13450 7050 13300 7050
+Text Label 13450 7050 0    50   ~ 0
+P2+
+Text HLabel 13300 7150 0    50   Input ~ 0
+P2-
+Wire Wire Line
+	13450 7150 13300 7150
+Text Label 13450 7150 0    50   ~ 0
+P2-
+Text Label 13650 8650 0    50   ~ 0
+P2+
+Text Label 13650 8550 0    50   ~ 0
+P1+
+Wire Wire Line
+	13650 8650 13900 8650
+Wire Wire Line
+	13650 8550 13900 8550
+Wire Wire Line
+	13900 8550 13900 8650
+Wire Wire Line
+	13900 8650 14200 8650
+Connection ~ 13900 8650
+Text Label 14200 8650 2    50   ~ 0
+12V_DL
 $EndSCHEMATC

Commit message: Restructure into three boards
Parts:
- removed C? (x10): 10n, symbol cusf-kicad:C
- removed C? (x5): 1u, symbol cusf-kicad:C
- removed C? (x4): 100n, agg:0402, symbol cusf-kicad:C
- removed C? (x4): 82n, symbol cusf-kicad:C
- removed C? (x4): 8n2, symbol cusf-kicad:C
- removed C? (x16): 100n, symbol cusf-kicad:C
- removed D? (x8): ESD_DIODE, cusf:0402, symbol cusf-kicad:ESD_DIODE
- removed IC?: ADP3335, cusf:MSOP-8, symbol cusf-kicad:ADP3335
- removed IC? (x12): AD8656, cusf:MSOP-8, symbol cusf-kicad:AD8656
- removed IC? (x4): AD8495, cusf:MSOP-8, symbol cusf-kicad:AD8495
- removed R? (x6): 6k04, symbol cusf-kicad:R
- removed R? (x2): 562R, symbol cusf-kicad:R
- removed R? (x2): 17k8, symbol cusf-kicad:R
- removed R? (x12): 1k, symbol cusf-kicad:R
- removed R? (x4): 8k87, symbol cusf-kicad:R
- removed R? (x4): 31k6, symbol cusf-kicad:R
- removed R? (x4): 2k94, symbol cusf-kicad:R
- removed R? (x4): 95k3, symbol cusf-kicad:R
- added C? (x4): 100n, agg:0402, symbol cusf-kicad:C
- added D? (x3): ESD_DIODE, cusf:0402, symbol cusf-kicad:ESD_DIODE
- added J?: USB, symbol cusf-kicad:CONN_01x04
- added R?: 1k, symbol cusf-kicad:R
Connections:
- net labels added: FLASH_CS, FLASH_MISO, FLASH_MOSI, FLASH_SCK, OTG_HS_D+, OTG_HS_D-
- net labels removed: 12V_DL, 3V3, AGND, AVCC, P1+, P1-, P2+, P2-, PRESSURE1, PRESSURE2, SPI1_CS, SPI1_MISO, SPI1_MOSI, SPI1_SCK, TEMP1+, TEMP1-, TEMP2+, TEMP2-, TEMP3+, TEMP3-, TEMP4+, TEMP4-, TEMP_INT
- wire segments 615 -> 188
- no-connect marks 24 -> 32
Other:
- note added: "FLASH STORAGE"
- note added: "USB OTG HS"
- note removed: "- 150R current shunt required for\n 0.6v to 3v @ 4mA to 20mA\n\n- Pressure sensors are highest rate so\n should be connected to ADC123_x\n\n- All analog circuitry should be connected\n between VDD_A and AGND. AGND should\n be a separate sground plane connected to\n GND by a single trace wide enough to sink\n all of AGND"
- note removed: "Analog Supply (500mA @ 3v3)"
- note removed: "NOTES:"
- note removed: "PRESSURE FRONT-ENDS"
- note removed: "SPI FLASH"
- note removed: "THERMOCOUPLE FRONT-ENDS"
- moved on the sheet: C?, IC?, R?, U?
